Commit message: fixing world frame and laser scanner and spawning two robots in gazebo

File: xacro/barista_robot_model.urdf.xacro (robot description, xacro)
@@ -5,10 +5,13 @@
 <xacro:include filename="$(find barista_robot_description)/xacro/standoff.xacro" />
 <xacro:include filename="$(find barista_robot_description)/xacro/cup_holder_tray.xacro" />
-<xacro:include filename="$(find barista_robot_description)/xacro/laser_scanner.xacro" />
+<xacro:include filename="$(find barista_robot_description)/xacro/laser_scanner_old.xacro" />
   <material name="red">
       <color rgba="1.0 0.0 0.0 1"/>
   </material>
-  <material name="green">
+  <material name="green_light">
       <color rgba="0.0 1.0 0.0 1"/>
+  </material>
+  <material name="green_dark">
+    <color rgba="0.0 0.5 0.0 1"/>
   </material>
   <material name="blue">
@@ -20,4 +23,7 @@
   <material name="white">
       <color rgba="1.0 1.0 1.0 1"/>
+  </material>
+  <material name="barista_bot_blue">
+      <color rgba="0.088656 0.428691 0.491021 1"/>
   </material>
   <link name="base_link">
@@ -50,38 +56,51 @@
         <material>Gazebo/Red</material>
   </gazebo>
-<xacro:standoff rod_num="rod_1" />
-      <joint name="rod_1_joint" type="fixed">
-        <parent link="base_link"/>
-        <child link="rod_1"/>
-        <origin rpy="0 0 0" xyz="0.130 0.05 0.185" />
-      </joint>
-<xacro:standoff rod_num="rod_2" />
-      <joint name="rod_2_joint" type="fixed">
-        <parent link="base_link"/>
-        <child link="rod_2"/>
-        <origin xyz="0.130 -0.05 0.185" rpy="0 0 0"/>
-      </joint>
-<xacro:standoff rod_num="rod_3" />
-      <joint name="rod_3_joint" type="fixed">
-        <parent link="base_link"/>
-        <child link="rod_3"/>
-        <origin xyz="-0.130 0.05 0.185" rpy="0 0 0"/>
-      </joint>
-<xacro:standoff rod_num="rod_4" />
-      <joint name="rod_4_joint" type="fixed">
-        <parent link="base_link"/>
-        <child link="rod_4"/>
-        <origin xyz="-0.130 -0.05 0.185" rpy="0 0 0"/>
-      </joint>
+  <xacro:standoff rod_name="rod_1" />
+  <xacro:standoff rod_name="rod_2" />
+  <xacro:standoff rod_name="rod_3" />
+  <xacro:standoff rod_name="rod_4" />
+  <joint name="rod_1_joint" type="fixed">
+    <parent link="base_link"/>
+    <child link="rod_1"/>
+    <origin rpy="0 0 0" xyz="0.130 0.05 0.185" />
+  </joint>
+  <gazebo reference="rod_1">
+        <material>Gazebo/White</material>
+  </gazebo>
+  <joint name="rod_2_joint" type="fixed">
+    <parent link="base_link"/>
+    <child link="rod_2"/>
+    <origin xyz="0.130 -0.05 0.185" rpy="0 0 0"/>
+  </joint>
+  <gazebo reference="rod_2">
+        <material>Gazebo/White</material>
+  </gazebo>
+  <joint name="rod_3_joint" type="fixed">
+    <parent link="base_link"/>
+    <child link="rod_3"/>
+    <origin xyz="-0.130 0.05 0.185" rpy="0 0 0"/>
+  </joint>
+  <gazebo reference="rod_3">
+        <material>Gazebo/White</material>
+  </gazebo>
+  <joint name="rod_4_joint" type="fixed">
+    <parent link="base_link"/>
+    <child link="rod_4"/>
+    <origin xyz="-0.130 -0.05 0.185" rpy="0 0 0"/>
+  </joint>
+  <gazebo reference="rod_4">
+        <material>Gazebo/White</material>
+  </gazebo>
 <xacro:cup_holder_tray cup_name="cupholder_link" />
-    <joint name="cupholder_joint" type="fixed">
-        <parent link="base_link"/>
-        <child link="cupholder_link"/>
-        <origin xyz="0 0 0.330" rpy="0 0 0"/>
-    </joint>
-    <gazebo reference="cupholder_link">
-        <material>Gazebo/Red</material>
-    </gazebo>
-<xacro:wheel wheel_name="left_wheel" />
+<joint name="cupholder_joint" type="fixed">
+  <parent link="base_link"/>
+  <child link="cupholder_link"/>
+  <origin xyz="0 0 0.330" rpy="0 0 0"/>
+</joint>
+<gazebo reference="cupholder_link">
+    <material>Gazebo/Red</material>
+</gazebo>
+  <xacro:wheel wheel_name="left_wheel" />
+  <xacro:wheel wheel_name="right_wheel" />
   <joint name="joint_left_wheel" type="fixed">
     <origin rpy="0 0 0" xyz="0 0.15 -0.0775"/>
@@ -92,5 +111,4 @@
     <joint_properties damping="1.0" friction="1.0"/>
   </joint>
-<xacro:wheel wheel_name="right_wheel" />
   <joint name="joint_right_wheel" type="fixed">
     <origin rpy="0 0 0" xyz="0 -0.15 -0.0775"/>
@@ -101,5 +119,19 @@
     <joint_properties damping="1.0" friction="1.0"/>
   </joint>
-<xacro:caster pos="front" />
+  <gazebo reference="left_wheel">
+    <kp>10000000000000.0</kp>
+    <kd>10000000000000.0</kd>
+    <mu1>10.0</mu1>
+    <mu2>10.0</mu2>
+    <material>Gazebo/Black</material>
+  </gazebo>
+  <gazebo reference="right_wheel">
+    <kp>10000000000000.0</kp>
+    <kd>10000000000000.0</kd>
+    <mu1>10.0</mu1>
+    <mu2>10.0</mu2>
+    <material>Gazebo/Black</material>
+  </gazebo>
+<xacro:caster posi="front" />
   <joint name="front_yaw_joint" type="fixed">
     <origin rpy="0 0 0" xyz="0.10 0 -0.0770" />
@@ -122,5 +154,5 @@
   </joint>
   <gazebo reference="front_roll_link">
-        <material>Gazebo/Red</material>
+        <material>Gazebo/Blue</material>
   </gazebo>
   <joint name="front_pitch_joint" type="fixed">
@@ -133,11 +165,11 @@
   </joint>
   <gazebo reference="front_pitch_link">
-    <kp>1000000000.0</kp>
-    <kd>1000000000.0</kd>
+    <kp>10000000.0</kp>
+    <kd>10000000.0</kd>
     <mu1>0.5</mu1>
     <mu2>0.5</mu2>
-    <material>Gazebo/White</material>
-  </gazebo>
-<xacro:caster pos="back" />
+    <material>Gazebo/Black</material>
+  </gazebo>
+<xacro:caster posi="back" />
   <joint name="back_yaw_joint" type="fixed">
     <origin rpy="0 0 0" xyz="-0.10 0 -0.0770" />
@@ -160,5 +192,5 @@
   </joint>
   <gazebo reference="back_roll_link">
-        <material>Gazebo/Red</material>
+        <material>Gazebo/Blue</material>
   </gazebo>
   <joint name="back_pitch_joint" type="fixed">
@@ -175,7 +207,7 @@
     <mu1>0.5</mu1>
     <mu2>0.5</mu2>
-    <material>Gazebo/White</material>
-  </gazebo>
-<xacro:laser_scanner include_laser="$(arg include_laser)"/>
+    <material>Gazebo/Blue</material>
+  </gazebo>
+<xacro:laser_scanner include_laser="True" />
   <!-- Differential drive -->
   <gazebo>
@@ -185,6 +217,6 @@
       <right_joint>joint_right_wheel</right_joint>
       <!-- kinematics -->
-      <wheel_separation>0.1</wheel_separation>
-      <wheel_diameter>0.07</wheel_diameter>
+      <wheel_separation>0.3</wheel_separation>
+      <wheel_diameter>0.0704</wheel_diameter>
       <!-- limits -->
       <max_wheel_torque>1.0</max_wheel_torque>

File: xacro/barista_two_robot_model_.urdf.xacro (robot description, xacro)
@@ -7,13 +7,23 @@
 <xacro:include filename="$(find barista_robot_description)/xacro/laser_scanner.xacro" />
 <xacro:property name="robot_name" value="$(arg robot_name)"/>
+<xacro:property name="gazebo_color" value="$(arg gazebo_color)" />
   <material name="red">
       <color rgba="1.0 0.0 0.0 1"/>
   </material>
-  <material name="green">
+  <material name="rick_color">
+      <color rgba="1.0 0.0 0.0 1"/>
+  </material>
+  <material name="green_light">
       <color rgba="0.0 1.0 0.0 1"/>
+  </material>
+  <material name="green_dark">
+    <color rgba="0.0 0.5 0.0 1"/>
   </material>
   <material name="blue">
       <color rgba="0.0 0.0 1.0 1"/>
   </material>
+    <material name="morty_color">
+      <color rgba="0.0 0.0 1.0 1"/>
+  </material>
   <material name="black">
       <color rgba="0.0 0.0 0.0 1"/>
@@ -22,6 +32,10 @@
       <color rgba="1.0 1.0 1.0 1"/>
   </material>
+  <material name="barista_bot_blue">
+      <color rgba="0.088656 0.428691 0.491021 1"/>
+  </material>
   <link name="base_link">
   </link>
+<material name="rick" script="model://barista_robot_description/materials/rick.material"/>
   <!-- Body -->
   <link name="chassis">
@@ -30,5 +44,5 @@
         <cylinder length="0.155" radius="0.178"/>
       </geometry>
-      <material name="red"/>
+        <material name="${robot_name}_color"/>
     </visual>
     <collision>
@@ -48,42 +62,55 @@
     <child link="chassis" />
   </joint>
-    <gazebo reference="chassis">
-        <material>Gazebo/Red</material>
-  </gazebo>
-<xacro:standoff rod_num="rod_1" />
-      <joint name="rod_1_joint" type="fixed">
-        <parent link="base_link"/>
-        <child link="rod_1"/>
-        <origin rpy="0 0 0" xyz="0.130 0.05 0.185" />
-      </joint>
-<xacro:standoff rod_num="rod_2" />
-      <joint name="rod_2_joint" type="fixed">
-        <parent link="base_link"/>
-        <child link="rod_2"/>
-        <origin xyz="0.130 -0.05 0.185" rpy="0 0 0"/>
-      </joint>
-<xacro:standoff rod_num="rod_3" />
-      <joint name="rod_3_joint" type="fixed">
-        <parent link="base_link"/>
-        <child link="rod_3"/>
-        <origin xyz="-0.130 0.05 0.185" rpy="0 0 0"/>
-      </joint>
-<xacro:standoff rod_num="rod_4" />
-      <joint name="rod_4_joint" type="fixed">
-        <parent link="base_link"/>
-        <child link="rod_4"/>
-        <origin xyz="-0.130 -0.05 0.185" rpy="0 0 0"/>
-      </joint>
+  <gazebo reference="chassis">
+    <material>${gazebo_color}</material>
+  </gazebo>
+  <xacro:standoff rod_name="rod_1" />
+  <xacro:standoff rod_name="rod_2" />
+  <xacro:standoff rod_name="rod_3" />
+  <xacro:standoff rod_name="rod_4" />
+  <joint name="rod_1_joint" type="fixed">
+    <parent link="base_link"/>
+    <child link="rod_1"/>
+    <origin rpy="0 0 0" xyz="0.130 0.05 0.185" />
+  </joint>
+  <gazebo reference="rod_1">
+        <material>Gazebo/White</material>
+  </gazebo>
+  <joint name="rod_2_joint" type="fixed">
+    <parent link="base_link"/>
+    <child link="rod_2"/>
+    <origin xyz="0.130 -0.05 0.185" rpy="0 0 0"/>
+  </joint>
+  <gazebo reference="rod_2">
+        <material>Gazebo/White</material>
+  </gazebo>
+  <joint name="rod_3_joint" type="fixed">
+    <parent link="base_link"/>
+    <child link="rod_3"/>
+    <origin xyz="-0.130 0.05 0.185" rpy="0 0 0"/>
+  </joint>
+  <gazebo reference="rod_3">
+        <material>Gazebo/White</material>
+  </gazebo>
+  <joint name="rod_4_joint" type="fixed">
+    <parent link="base_link"/>
+    <child link="rod_4"/>
+    <origin xyz="-0.130 -0.05 0.185" rpy="0 0 0"/>
+  </joint>
+  <gazebo reference="rod_4">
+        <material>Gazebo/White</material>
+  </gazebo>
 <xacro:cup_holder_tray cup_name="cupholder_link" />
-    <joint name="cupholder_joint" type="fixed">
-        <parent link="base_link"/>
-        <child link="cupholder_link"/>
-        <origin xyz="0 0 0.330" rpy="0 0 0"/>
-    </joint>
-    <gazebo reference="cupholder_link">
-        <material>Gazebo/Red</material>
-    </gazebo>
-<xacro:wheel wheel_name="left_wheel" />
-  <joint name="joint_left_wheel" type="fixed">
+<joint name="cupholder_joint" type="fixed">
+  <parent link="base_link"/>
+  <child link="cupholder_link"/>
+  <origin xyz="0 0 0.330" rpy="0 0 0"/>
+</joint>
+<gazebo reference="cupholder_link">
+    <material>${gazebo_color}</material>
+</gazebo>
+  <xacro:wheel wheel_name="left_wheel" />
+  <xacro:wheel wheel_name="right_wheel" />
+  <joint name="joint_left_wheel" type="continuous">
     <origin rpy="0 0 0" xyz="0 0.15 -0.0775"/>
     <child link="left_wheel"/>
@@ -93,6 +120,5 @@
     <joint_properties damping="1.0" friction="1.0"/>
   </joint>
-<xacro:wheel wheel_name="right_wheel" />
-  <joint name="joint_right_wheel" type="fixed">
+  <joint name="joint_right_wheel" type="continuous">
     <origin rpy="0 0 0" xyz="0 -0.15 -0.0775"/>
     <child link="right_wheel"/>
@@ -102,5 +128,19 @@
     <joint_properties damping="1.0" friction="1.0"/>
   </joint>
-<xacro:caster pos="front" />
+  <gazebo reference="left_wheel">
+    <kp>10000000000000.0</kp>
+    <kd>10000000000000.0</kd>
+    <mu1>10.0</mu1>
+    <mu2>10.0</mu2>
+    <material>Gazebo/Black</material>
+  </gazebo>
+  <gazebo reference="right_wheel">
+    <kp>10000000000000.0</kp>
+    <kd>10000000000000.0</kd>
+    <mu1>10.0</mu1>
+    <mu2>10.0</mu2>
+    <material>Gazebo/Black</material>
+  </gazebo>
+<xacro:caster posi="front" />
   <joint name="front_yaw_joint" type="fixed">
     <origin rpy="0 0 0" xyz="0.10 0 -0.0770" />
@@ -123,5 +163,5 @@
   </joint>
   <gazebo reference="front_roll_link">
-        <material>Gazebo/Red</material>
+        <material>Gazebo/Blue</material>
   </gazebo>
   <joint name="front_pitch_joint" type="fixed">
@@ -134,11 +174,11 @@
   </joint>
   <gazebo reference="front_pitch_link">
-    <kp>1000000000.0</kp>
-    <kd>1000000000.0</kd>
+    <kp>10000000.0</kp>
+    <kd>10000000.0</kd>
     <mu1>0.5</mu1>
     <mu2>0.5</mu2>
-    <material>Gazebo/White</material>
-  </gazebo>
-<xacro:caster pos="back" />
+    <material>Gazebo/Black</material>
+  </gazebo>
+<xacro:caster posi="back" />
   <joint name="back_yaw_joint" type="fixed">
     <origin rpy="0 0 0" xyz="-0.10 0 -0.0770" />
@@ -161,5 +201,5 @@
   </joint>
   <gazebo reference="back_roll_link">
-        <material>Gazebo/Red</material>
+        <material>Gazebo/Blue</material>
   </gazebo>
   <joint name="back_pitch_joint" type="fixed">
@@ -176,9 +216,9 @@
     <mu1>0.5</mu1>
     <mu2>0.5</mu2>
-    <material>Gazebo/White</material>
-  </gazebo>
-<xacro:laser_scanner include_laser="$(arg include_laser)" robot_name="${robot_name}"/>
-<gazebo>
-    <plugin name="box_bot_joint_state" filename="libgazebo_ros_joint_state_publisher.so">
+    <material>Gazebo/Blue</material>
+  </gazebo>
+  <xacro:laser_scanner include_laser="$(arg include_laser)" robot_name="${robot_name}" />
+    <gazebo>
+    <plugin name="joint_state" filename="libgazebo_ros_joint_state_publisher.so">
       <ros>
           <namespace>/${robot_name}</namespace>
@@ -203,6 +243,6 @@
       <right_joint>joint_right_wheel</right_joint>
       <!-- kinematics -->
-      <wheel_separation>0.1</wheel_separation>
-      <wheel_diameter>0.07</wheel_diameter>
+      <wheel_separation>0.3</wheel_separation>
+      <wheel_diameter>0.0704</wheel_diameter>
       <!-- limits -->
       <max_wheel_torque>1.0</max_wheel_torque>
@@ -211,6 +251,10 @@
       <publish_odom>true</publish_odom>
       <publish_odom_tf>true</publish_odom_tf>
-      <odometry_frame>odom</odometry_frame>
-      <robot_base_frame>base_link</robot_base_frame>
+      <odometry_frame>${robot_name}/odom</odometry_frame>
+      <robot_base_frame>${robot_name}/base_link</robot_base_frame>
+        <ros>
+            <namespace>/${robot_name}</namespace>
+            <remapping>~/out:=cmd_vel</remapping>
+        </ros>
     </plugin>
   </gazebo>

File: xacro/caster.xacro (robot description, xacro)
@@ -3,6 +3,6 @@
   <xacro:property name="caster_length" value="0.01" />
   <xacro:property name="caster_radius" value="0.035" />
-<xacro:macro name="caster" params="pos">
-  <link name="${pos}_yaw_link">
+<xacro:macro name="caster" params="posi">
+  <link name="${posi}_yaw_link">
     <visual>
         <origin rpy="0 1.5707 1.5707" xyz="0 0 0"/>
@@ -19,5 +19,5 @@
     </collision>
   </link>
-  <link name="${pos}_roll_link">
+  <link name="${posi}_roll_link">
       <visual>
         <origin rpy="0 1.5707 1.5707" xyz="0 0 0"/>
@@ -34,5 +34,5 @@
     </collision>
   </link>
-  <link name="${pos}_pitch_link">
+  <link name="${posi}_pitch_link">
     <visual>
       <origin rpy="0 1.5707 1.5707" xyz="0 0 0"/>
@@ -40,5 +40,5 @@
         <sphere radius="${caster_radius}"/>
       </geometry>
-      <material name="white"/>
+      <material name="black"/>
     </visual>
     <collision>

File: xacro/cup_holder_tray.xacro (robot description, xacro)
@@ -1,6 +1,6 @@
 <?xml version="1.0"?>
 <robot name="cup_holder_tray"  xmlns:xacro="http://ros.org/wiki/xacro">
-  <xacro:property name="holder_length" value="0.09" />
-  <xacro:property name="holder_radius" value="0.16" />
+  <xacro:property name="cup_length" value="0.09" />
+  <xacro:property name="cup_radius" value="0.16" />
 <xacro:macro name="cup_holder_tray" params="cup_name">
   <link name="${cup_name}">
@@ -8,5 +8,5 @@
     <origin xyz="0 0 0" rpy="0 0 0"/>
     <geometry>
-      <cylinder length="${holder_length}" radius="${holder_radius}"/>
+      <cylinder length="${cup_length}" radius="${cup_radius}"/>
     </geometry>
   </visual>
@@ -14,5 +14,5 @@
     <origin xyz="0 0 0" rpy="0 0 0"/>
     <geometry>
-      <cylinder length="${holder_length}" radius="${holder_radius}"/>
+      <cylinder length="${cup_length}" radius="${cup_radius}"/>
     </geometry>
   </collision>
@@ -23,6 +23,4 @@
     </inertial>
   </link>
-<xacro:if value="${cup_name == 'cupholder_link'}">
-</xacro:if>
 </xacro:macro>
 </robot>

File: xacro/laser_scanner_old.xacro (robot description, xacro)
@@ -1,19 +1,20 @@
 <?xml version="1.0"?>
 <robot xmlns:xacro="http://ros.org/wiki/xacro">
-  <xacro:macro name="laser_scanner" params="robot_name include_laser:=true">
+  <xacro:macro name="laser_scanner" params="include_laser:=true">
     <xacro:if value="${include_laser}">
-      <link name="lidar">
-          <visual>
-          <origin rpy="0 0 0" xyz="0.0 0 -0.055" />
-              <geometry>
-                  <mesh filename="package://barista_robot_description/meshes/hokuyo_urg_04lx.dae"/>
-              </geometry>
-          </visual>
-      </link>
-      <joint name="lidar_joint" type="fixed">
-          <origin rpy="0 0 0" xyz="0.120 0 0.130" />
-          <parent link="chassis" />
-          <child link="lidar" />
-      </joint>
+    <link name="lidar">
+        <visual>
+        <origin rpy="0 0 0" xyz="0 0 -0.055" />
+            <geometry>
+                <mesh filename="package://barista_robot_description/meshes/hokuyo_urg_04lx.dae"/>
+            </geometry>
+      <material name="black"/>
+        </visual>
+    </link>
+    <joint name="lidar_joint" type="fixed">
+        <origin rpy="0 0 0" xyz="0.120 0 0.130" />
+        <parent link="base_link" />
+        <child link="lidar" />
+    </joint>
       <gazebo reference="lidar">
           <material>Gazebo/Black</material>
@@ -40,8 +41,5 @@
           <update_rate>50.0</update_rate>
           <plugin name="laser" filename="libgazebo_ros_ray_sensor.so">
-            <frame_name>${robot_name}/base_link</frame_name>
-            <topic_name>${robot_name}/scan</topic_name>
             <ros>
-              <namespace>${robot_name}</namespace>
               <remapping>~/out:=scan</remapping>
             </ros>

File: xacro/standoff.xacro (robot description, xacro)
@@ -1,12 +1,12 @@
 <?xml version="1.0"?>
 <robot name="standoff"  xmlns:xacro="http://ros.org/wiki/xacro">
-  <xacro:property name="rlength" value="0.22" />
-  <xacro:property name="rradius" value="0.01" />
-<xacro:macro name="standoff" params="rod_num">
-  <link name="${rod_num}">
+  <xacro:property name="rod_length" value="0.22" />
+  <xacro:property name="rod_radius" value="0.01" />
+<xacro:macro name="standoff" params="rod_name">
+  <link name="${rod_name}">
     <visual>
       <origin xyz="0 0 0" rpy="0 0 0"/>
       <geometry>
-        <cylinder length="${rlength}" radius="${rradius}"/>
+        <cylinder length="${rod_length}" radius="${rod_radius}"/>
       </geometry>
       <material name="white"/>
@@ -15,5 +15,5 @@
       <origin xyz="0 0 0" rpy="0 0 0"/>
       <geometry>
-        <cylinder length="${rlength}" radius="${rradius}"/>
+        <cylinder length="${rod_length}" radius="${rod_radius}"/>
       </geometry>
     </collision>
@@ -24,7 +24,4 @@
     </inertial>
   </link>
-    <gazebo reference="${rod_num}">
-      <material>Gazebo/White</material>
-    </gazebo>
 </xacro:macro>
 </robot>

File: xacro/wheel.xacro (robot description, xacro)
@@ -1,6 +1,6 @@
 <?xml version="1.0"?>
 <robot name="wheel"  xmlns:xacro="http://ros.org/wiki/xacro">
-  <xacro:property name="wheelradius" value="0.0352" />
-  <xacro:property name="wheelwidth" value="0.0206" />
+  <xacro:property name="wheel_radius" value="0.0352" />
+  <xacro:property name="wheel_width" value="0.0206" />
 <xacro:macro name="wheel" params="wheel_name">
   <link name="${wheel_name}">
@@ -8,12 +8,11 @@
         <origin rpy="0 1.5707 1.5707" xyz="0 0 0"/>
         <geometry>
-          <cylinder length="${wheelwidth}" radius="${wheelradius}"/>
+          <cylinder length="${wheel_width}" radius="${wheel_radius}"/>
         </geometry>
-        <material name="black" />
       </visual>
       <collision>
         <origin rpy="0 1.5707 1.5707" xyz="0 0 0"/>
         <geometry>
-          <cylinder length="${wheelwidth}" radius="${wheelradius}"/>
+          <cylinder length="${wheel_width}" radius="${wheel_radius}"/>
         </geometry>
       </collision>
@@ -24,11 +23,4 @@
     </inertial>
   </link>
-  <gazebo reference="${wheel_name}">
-    <kp>10000000000000.0</kp>
-    <kd>10000000000000.0</kd>
-    <mu1>10.0</mu1>
-    <mu2>10.0</mu2>
-    <material>Gazebo/Black</material>
-  </gazebo>
 </xacro:macro>
 </robot>
