Commit message: Adding gazebo plugins

File: urdf/barista_robot_model.urdf (robot description, URDF)
Before this commit: robot box_bot, 15 links, 14 joints
Links:
- added link lidar; visual mesh filename=package://barista_robot_description/meshes/hokuyo_urg_04lx.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
Joints:
- added joint lidar_joint: type fixed, parent base_link, child lidar, origin xyz=0 0 0.0775 rpy=0 0 0
- joint back_pitch_joint: type continuous -> fixed
- joint back_roll_joint: type continuous -> fixed
- joint back_yaw_joint: type continuous -> fixed
- joint front_pitch_joint: type continuous -> fixed
- joint front_roll_joint: type continuous -> fixed
- joint front_yaw_joint: type continuous -> fixed

Commit message: modified rviz2 and xacro files

File: urdf/barista_robot_model.urdf (robot description, URDF)
Before this commit: robot barista_bot, 16 links, 15 joints
Links:
- link back_pitch_link: geometry collision cylinder length=0.015 radius=0.0352; visual sphere radius=0.0352
- link back_roll_link: geometry collision cylinder length=0.015 radius=0.0352; visual cylinder length=0.015 radius=0.0352
- link back_yaw_link: geometry collision cylinder length=0.015 radius=0.0352; visual cylinder length=0.015 radius=0.0352
- link front_pitch_link: geometry collision cylinder length=0.015 radius=0.0352; visual sphere radius=0.0352
- link front_roll_link: geometry collision cylinder length=0.015 radius=0.0352; visual cylinder length=0.015 radius=0.0352
- link front_yaw_link: geometry collision cylinder length=0.015 radius=0.0352; visual cylinder length=0.015 radius=0.0352

File: xacro/barista_robot_model.urdf.xacro (robot description, xacro)
@@ -2,4 +2,5 @@
 <robot name="barista_bot" xmlns:xacro="http://ros.org/wiki/xacro">
 <xacro:include filename="$(find barista_robot_description)/xacro/wheel.xacro" />
+<xacro:include filename="$(find barista_robot_description)/xacro/caster.xacro" />
 <xacro:include filename="$(find barista_robot_description)/xacro/standoff.xacro" />
 <xacro:include filename="$(find barista_robot_description)/xacro/cup_holder_tray.xacro" />
@@ -50,26 +51,52 @@
   </gazebo>
 <xacro:standoff rod_num="rod_1" />
+      <joint name="rod_1_joint" type="fixed">
+        <parent link="base_link"/>
+        <child link="rod_1"/>
+        <origin rpy="0 0 0" xyz="0.130 0.05 0.185" />
+      </joint>
 <xacro:standoff rod_num="rod_2" />
+      <joint name="rod_2_joint" type="fixed">
+        <parent link="base_link"/>
+        <child link="rod_2"/>
+        <origin xyz="0.130 -0.05 0.185" rpy="0 0 0"/>
+      </joint>
 <xacro:standoff rod_num="rod_3" />
+      <joint name="rod_3_joint" type="fixed">
+        <parent link="base_link"/>
+        <child link="rod_3"/>
+        <origin xyz="-0.130 0.05 0.185" rpy="0 0 0"/>
+      </joint>
 <xacro:standoff rod_num="rod_4" />
+      <joint name="rod_4_joint" type="fixed">
+        <parent link="base_link"/>
+        <child link="rod_4"/>
+        <origin xyz="-0.130 -0.05 0.185" rpy="0 0 0"/>
+      </joint>
 <xacro:cup_holder_tray cup_name="cupholder_link" />
+    <joint name="cupholder_joint" type="fixed">
+        <parent link="base_link"/>
+        <child link="cupholder_link"/>
+        <origin xyz="0 0 0.330" rpy="0 0 0"/>
+    </joint>
 <xacro:wheel wheel_name="left_wheel" />
+  <joint name="joint_left_wheel" type="fixed">
+    <origin rpy="0 0 0" xyz="0 0.15 -0.0775"/>
+    <child link="left_wheel"/>
+    <parent link="base_link"/>
+    <axis rpy="0 0 0" xyz="0 1 0"/>
+    <limit effort="1000" velocity="100"/>
+    <joint_properties damping="1.0" friction="1.0"/>
+  </joint>
 <xacro:wheel wheel_name="right_wheel" />
-  <!-- Caster Wheel Front -->
-  <link name="front_yaw_link">
-    <visual>
-        <origin rpy="0 1.5707 1.5707" xyz="0 0 0"/>
-        <geometry>
-          <cylinder length="0.015" radius="0.025"/>
-        </geometry>
-        <material name="blue"/>
-      </visual>
-    <collision>
-      <origin rpy="0 1.5707 1.5707" xyz="0 0 0" />
-      <geometry>
-            <cylinder length="0.015" radius="0.025"/>
-      </geometry>
-    </collision>
-  </link>
+  <joint name="joint_right_wheel" type="fixed">
+    <origin rpy="0 0 0" xyz="0 -0.15 -0.0775"/>
+    <child link="right_wheel"/>
+    <parent link="base_link"/>
+    <axis rpy="0 0 0" xyz="0 1 0"/>
+    <limit effort="1000" velocity="100"/>
+    <joint_properties damping="1.0" friction="1.0"/>
+  </joint>
+<xacro:caster pos="front" />
   <joint name="front_yaw_joint" type="fixed">
     <origin rpy="0 0 0" xyz="0.10 0 -0.0770" />
@@ -83,19 +110,4 @@
         <material>Gazebo/Blue</material>
   </gazebo>
-  <link name="front_roll_link">
-      <visual>
-        <origin rpy="0 1.5707 1.5707" xyz="0 0 0"/>
-        <geometry>
-          <cylinder length="0.015" radius="0.025"/>
-        </geometry>
-        <material name="red"/>
-      </visual>
-      <collision>
-      <origin rpy="0 1.5707 1.5707" xyz="0 0 0" />
-      <geometry>
-        <cylinder length="0.015" radius="0.025"/>
-      </geometry>
-     </collision>
-  </link>
   <joint name="front_roll_joint" type="fixed">
     <origin rpy="0 0 0" xyz="0 0 0" />
@@ -109,19 +121,4 @@
         <material>Gazebo/Red</material>
   </gazebo>
-  <link name="front_pitch_link">
-    <visual>
-      <origin rpy="0 1.5707 1.5707" xyz="0 0 0"/>
-      <geometry>
-        <sphere radius="0.025"/>
-      </geometry>
-      <material name="white"/>
-    </visual>
-    <collision>
-      <origin rpy="0 1.5707 1.5707" xyz="0 0 0" />
-      <geometry>
-        <cylinder length="0.015" radius="0.025"/>
-      </geometry>
-    </collision>
-  </link>
   <joint name="front_pitch_joint" type="fixed">
     <origin rpy="0 0 0" xyz="0 0 0" />
@@ -133,26 +130,11 @@
   </joint>
   <gazebo reference="front_pitch_link">
-    <kp>10000000.0</kp>
-    <kd>10000000.0</kd>
+    <kp>1000000000.0</kp>
+    <kd>1000000000.0</kd>
     <mu1>0.5</mu1>
     <mu2>0.5</mu2>
     <material>Gazebo/White</material>
   </gazebo>
-<!-- Caster Wheel Back -->
-  <link name="back_yaw_link">
-    <visual>
-        <origin rpy="0 1.5707 1.5707" xyz="0 0 0"/>
-        <geometry>
-          <cylinder length="0.015" radius="0.025"/>
-        </geometry>
-        <material name="blue"/>
-      </visual>
-      <collision>
-      <origin rpy="0 1.5707 1.5707" xyz="0 0 0" />
-      <geometry>
-        <cylinder length="0.015" radius="0.025"/>
-      </geometry>
-    </collision>
-  </link>
+<xacro:caster pos="back" />
   <joint name="back_yaw_joint" type="fixed">
     <origin rpy="0 0 0" xyz="-0.10 0 -0.0770" />
@@ -166,19 +148,4 @@
         <material>Gazebo/Blue</material>
   </gazebo>
-  <link name="back_roll_link">
-      <visual>
-        <origin rpy="0 1.5707 1.5707" xyz="0 0 0"/>
-        <geometry>
-          <cylinder length="0.015" radius="0.025"/>
-        </geometry>
-        <material name="red"/>
-      </visual>
-      <collision>
-      <origin rpy="0 1.5707 1.5707" xyz="0 0 0" />
-      <geometry>
-        <cylinder length="0.015" radius="0.025"/>
-      </geometry>
-    </collision>
-  </link>
   <joint name="back_roll_joint" type="fixed">
     <origin rpy="0 0 0" xyz="0 0 0" />
@@ -192,19 +159,4 @@
         <material>Gazebo/Red</material>
   </gazebo>
-  <link name="back_pitch_link">
-    <visual>
-      <origin rpy="0 1.5707 1.5707" xyz="0 0 0"/>
-      <geometry>
-        <sphere radius="0.025"/>
-      </geometry>
-      <material name="white"/>
-    </visual>
-    <collision>
-      <origin rpy="0 1.5707 1.5707" xyz="0 0 0" />
-      <geometry>
-        <cylinder length="0.015" radius="0.025"/>
-      </geometry>
-    </collision>
-  </link>
   <joint name="back_pitch_joint" type="fixed">
     <origin rpy="0 0 0" xyz="0 0 0" />

File: xacro/cup_holder_tray.xacro (robot description, xacro)
@@ -1,6 +1,6 @@
 <?xml version="1.0"?>
 <robot name="cup_holder_tray"  xmlns:xacro="http://ros.org/wiki/xacro">
-  <xacro:property name="length" value="0.09" />
-  <xacro:property name="radius" value="0.16" />
+  <xacro:property name="holder_length" value="0.09" />
+  <xacro:property name="holder_radius" value="0.16" />
 <xacro:macro name="cup_holder_tray" params="cup_name">
   <link name="${cup_name}">
@@ -8,5 +8,5 @@
     <origin xyz="0 0 0" rpy="0 0 0"/>
     <geometry>
-      <cylinder length="${length}" radius="${radius}"/>
+      <cylinder length="${holder_length}" radius="${holder_radius}"/>
     </geometry>
   </visual>
@@ -14,5 +14,5 @@
     <origin xyz="0 0 0" rpy="0 0 0"/>
     <geometry>
-      <cylinder length="${length}" radius="${radius}"/>
+      <cylinder length="${holder_length}" radius="${holder_radius}"/>
     </geometry>
   </collision>
@@ -27,9 +27,4 @@
 </gazebo>
 <xacro:if value="${cup_name == 'cupholder_link'}">
-<joint name="cupholder_joint" type="fixed">
-  <parent link="base_link"/>
-  <child link="cupholder_link"/>
-  <origin xyz="0 0 0.330" rpy="0 0 0"/>
-</joint>
 </xacro:if>
 </xacro:macro>

File: xacro/standoff.xacro (robot description, xacro)
@@ -27,32 +27,4 @@
       <material>Gazebo/White</material>
     </gazebo>
-    <xacro:if value="${rod_num == 'rod_1'}">
-      <joint name="rod_1_joint" type="fixed">
-        <parent link="base_link"/>
-        <child link="rod_1"/>
-        <origin rpy="0 0 0" xyz="0.130 0.05 0.185" />
-      </joint>
-    </xacro:if>
-    <xacro:if value="${rod_num == 'rod_2'}">
-      <joint name="rod_2_joint" type="fixed">
-        <parent link="base_link"/>
-        <child link="rod_2"/>
-        <origin xyz="0.130 -0.05 0.185" rpy="0 0 0"/>
-      </joint>
-    </xacro:if>
-    <xacro:if value="${rod_num == 'rod_3'}">
-      <joint name="rod_3_joint" type="fixed">
-        <parent link="base_link"/>
-        <child link="rod_3"/>
-        <origin xyz="-0.130 0.05 0.185" rpy="0 0 0"/>
-      </joint>
-    </xacro:if>
-    <xacro:if value="${rod_num == 'rod_4'}">
-      <joint name="rod_4_joint" type="fixed">
-        <parent link="base_link"/>
-        <child link="rod_4"/>
-        <origin xyz="-0.130 -0.05 0.185" rpy="0 0 0"/>
-      </joint>
-    </xacro:if>
 </xacro:macro>
 </robot>

File: xacro/wheel.xacro (robot description, xacro)
@@ -1,6 +1,6 @@
 <?xml version="1.0"?>
 <robot name="wheel"  xmlns:xacro="http://ros.org/wiki/xacro">
-  <xacro:property name="wradius" value="0.0352" />
-  <xacro:property name="wwidth" value="0.0206" />
+  <xacro:property name="wheelradius" value="0.0352" />
+  <xacro:property name="wheelwidth" value="0.0206" />
 <xacro:macro name="wheel" params="wheel_name">
   <link name="${wheel_name}">
@@ -8,5 +8,5 @@
         <origin rpy="0 1.5707 1.5707" xyz="0 0 0"/>
         <geometry>
-          <cylinder length="${wwidth}" radius="${wradius}"/>
+          <cylinder length="${wheelwidth}" radius="${wheelradius}"/>
         </geometry>
         <material name="black" />
@@ -15,5 +15,5 @@
         <origin rpy="0 1.5707 1.5707" xyz="0 0 0"/>
         <geometry>
-          <cylinder length="${wwidth}" radius="${wradius}"/>
+          <cylinder length="${wheelwidth}" radius="${wheelradius}"/>
         </geometry>
       </collision>
@@ -31,24 +31,4 @@
     <material>Gazebo/Black</material>
   </gazebo>
-<xacro:if value="${wheel_name == 'left_wheel'}">
-  <joint name="joint_left_wheel" type="fixed">
-    <origin rpy="0 0 0" xyz="0 0.15 -0.0775"/>
-    <child link="left_wheel"/>
-    <parent link="base_link"/>
-    <axis rpy="0 0 0" xyz="0 1 0"/>
-    <limit effort="1000" velocity="100"/>
-    <joint_properties damping="1.0" friction="1.0"/>
-  </joint>
-</xacro:if>
-<xacro:if value="${wheel_name == 'right_wheel'}">
-  <joint name="joint_right_wheel" type="fixed">
-    <origin rpy="0 0 0" xyz="0 -0.15 -0.0775"/>
-    <child link="right_wheel"/>
-    <parent link="base_link"/>
-    <axis rpy="0 0 0" xyz="0 1 0"/>
-    <limit effort="1000" velocity="100"/>
-    <joint_properties damping="1.0" friction="1.0"/>
-  </joint>
-</xacro:if>
 </xacro:macro>
 </robot>

Commit message: spawning two barista robots

File: urdf/barista_robot_model.urdf (robot description, URDF)
Before this commit: robot barista_bot, 16 links, 15 joints
Joints:
- joint lidar_joint: origin xyz=0 0 0.0775 rpy=0 0 0 -> xyz=0.120 0 0.130 rpy=0 0 0

File: xacro/barista_tworobot_model.urdf.xacro (robot description, xacro)
@@ -6,4 +6,5 @@
 <xacro:include filename="$(find barista_robot_description)/xacro/cup_holder_tray.xacro" />
 <xacro:include filename="$(find barista_robot_description)/xacro/laser_scanner.xacro" />
+<xacro:property name="robot_name" value="$(arg robot_name)"/>
   <material name="red">
       <color rgba="1.0 0.0 0.0 1"/>
@@ -177,5 +178,22 @@
     <material>Gazebo/White</material>
   </gazebo>
-<xacro:laser_scanner include_laser="$(arg include_laser)"/>
+<xacro:laser_scanner include_laser="$(arg include_laser)" robot_name="${robot_name}"/>
+<gazebo>
+    <plugin name="box_bot_joint_state" filename="libgazebo_ros_joint_state_publisher.so">
+      <ros>
+          <namespace>/${robot_name}</namespace>
+          <remapping>~/out:=joint_states</remapping>
+      </ros>
+      <update_rate>30</update_rate>
+      <joint_name>joint_left_wheel</joint_name>
+      <joint_name>joint_right_wheel</joint_name>
+      <joint_name>front_yaw_joint</joint_name>
+      <joint_name>back_yaw_joint</joint_name>
+      <joint_name>front_roll_joint</joint_name>
+      <joint_name>back_roll_joint</joint_name>
+      <joint_name>front_pitch_joint</joint_name>
+      <joint_name>back_pitch_joint</joint_name>
+    </plugin>
+  </gazebo>
   <!-- Differential drive -->
   <gazebo>

File: xacro/cup_holder_tray.xacro (robot description, xacro)
@@ -23,7 +23,4 @@
     </inertial>
   </link>
-<gazebo reference="${cup_name}">
-    <material>Gazebo/Red</material>
-</gazebo>
 <xacro:if value="${cup_name == 'cupholder_link'}">
 </xacro:if>

File: xacro/laser_scanner.xacro (robot description, xacro)
@@ -1,9 +1,9 @@
 <?xml version="1.0"?>
 <robot name="laser_scanner"  xmlns:xacro="http://ros.org/wiki/xacro">
-<xacro:macro name="laser_scanner" params="include_laser:=true">
+<xacro:macro name="laser_scanner" params="robot_name include_laser:=true">
     <xacro:if value="${include_laser}">
     <link name="lidar">
         <visual>
-        <origin rpy="0 0 0" xyz="0 0 0" />
+        <origin rpy="0 0 0" xyz="0 0 -0.055" />
             <geometry>
                 <mesh filename="package://barista_robot_description/meshes/hokuyo_urg_04lx.dae"/>
@@ -13,5 +13,5 @@
     </link>
     <joint name="lidar_joint" type="fixed">
-        <origin rpy="0 0 0" xyz="0 0 0.0775" />
+        <origin rpy="0 0 0" xyz="0.120 0 0.130" />
         <parent link="base_link" />
         <child link="lidar" />
@@ -38,5 +38,8 @@
         <update_rate>100.0</update_rate>
         <plugin name="laser" filename="libgazebo_ros_ray_sensor.so">
+          <frame_name>$/base_link</frame_name>
+          <topic_name>$/scan</topic_name>
           <ros>
+            <namespace>${robot_name}</namespace>
             <remapping>~/out:=scan</remapping>
           </ros>

Commit message: Laserscan position and scale corrected again

File: urdf/barista_robot_model.urdf (robot description, URDF)
Before this commit: robot barista_bot, 16 links, 15 joints
Links:
- link lidar: geometry visual mesh filename=package://barista_robot_description/meshes/hokuyo_urg_04lx.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 scale=0.5 0.5 0.5
Joints:
- joint lidar_joint: origin xyz=0.120 0 0.130 rpy=0 0 0 -> xyz=0 0.130 0.08 rpy=0 0 0

File: xacro/laser_scanner.xacro (robot description, xacro)
@@ -5,12 +5,12 @@
       <link name="lidar">
           <visual>
-          <origin rpy="0 0 0" xyz="0.0 0 -0.055" />
+          <origin rpy="0 0 0" xyz="0 0 -0.0025" />
               <geometry>
-                  <mesh filename="package://barista_robot_description/meshes/hokuyo_urg_04lx.dae"/>
+                  <mesh filename="package://barista_robot_description/meshes/hokuyo_urg_04lx.dae" scale="1 1 1"/>
               </geometry>
           </visual>
       </link>
       <joint name="lidar_joint" type="fixed">
-          <origin rpy="0 0 0" xyz="0.120 0 0.130" />
+          <origin rpy="0 0 0" xyz="0 0.130 0.08" />
           <parent link="chassis" />
           <child link="lidar" />

File: xacro/laser_scanner_old.xacro (robot description, xacro)
@@ -5,7 +5,7 @@
     <link name="lidar">
         <visual>
-        <origin rpy="0 0 0" xyz="0 0 -0.055" />
+        <origin rpy="0 0 0" xyz="0 0 -0.0025" />
             <geometry>
-                <mesh filename="package://barista_robot_description/meshes/hokuyo_urg_04lx.dae"/>
+                <mesh filename="package://barista_robot_description/meshes/hokuyo_urg_04lx.dae" scale="1 1 1"/>
             </geometry>
       <material name="black"/>
@@ -13,5 +13,5 @@
     </link>
     <joint name="lidar_joint" type="fixed">
-        <origin rpy="0 0 0" xyz="0.120 0 0.130" />
+        <origin rpy="0 0 0" xyz="0 0.130 0.08" />
         <parent link="base_link" />
         <child link="lidar" />
